Commit message: Fixed angles

File: rcv_description/urdf/rcv.xacro (robot description, xacro)
@@ -31,12 +31,12 @@
   </joint>
   <joint name="velodyne_right_joint" type="fixed" >
-    <origin rpy="0 0 0"
-            xyz="0 0.7 0" />
+    <origin rpy="0 0 -1.57"
+            xyz="0 -0.7 0" />
     <parent link="sensor_board_link"/>
     <child link="velodyne_right"/>
   </joint>
   <joint name="velodyne_left_joint" type="fixed" >
-    <origin rpy="0 0 0"
-            xyz="0 -0.675 0" />
+    <origin rpy="0 0 1.57"
+            xyz="0 0.675 0" />
     <parent link="sensor_board_link"/>
     <child link="velodyne_left"/>
@@ -50,5 +50,5 @@
   <joint name="camera_left_joint" type="fixed" >
     <origin rpy="0 0 0"
-            xyz="0 -0.5 0" />
+            xyz="0 0.5 0" />
     <parent link="sensor_board_link"/>
     <child link="left_optical"/>
@@ -56,5 +56,5 @@
   <joint name="camera_right_joint" type="fixed" >
     <origin rpy="0 0 0"
-            xyz="0 0.5 0" />
+            xyz="0 -0.5 0" />
     <parent link="sensor_board_link"/>
     <child link="right_optical"/>

Commit message: Changed urdf

File: rcv_description/urdf/rcv.xacro (robot description, xacro)
@@ -44,7 +44,7 @@
   <joint name="trimble_joint" type="fixed" >
     <origin rpy="0 0 0"
-            xyz="0.06 0 0" />
-    <parent link="sensor_board_link"/>
-    <child link="trimble"/>
+            xyz="1.81 0 1.5" />
+    <parent link="trimble"/>
+    <child link="base_link"/>
   </joint>
   <joint name="camera_left_joint" type="fixed" >

Commit message: Added awesome mesh for the RCV, also changed urdf to match it

File: rcv_description/urdf/rcv.xacro (robot description, xacro)
@@ -8,5 +8,5 @@
   <!-- calibration data -->
   <!-- <xacro:include filename="$(find rcv_description)/urdf/rcv.xacro" /> -->
-  <!-- Base link is the actual robot body -->
+  <!-- Base link is the actual robot body, on the ground-->
   <link name="base_link">
     <collision>
@@ -24,4 +24,9 @@
   <link name="left_optical"/>
   <link name="right_optical"/>
+  <link name="flwheel"/>
+  <link name="frwheel"/>
+  <link name="rlwheel"/>
+  <link name="rrwheel"/>
+  <link name="imu"/>
   <joint name="base_sensor_board_joint" type="fixed" >
     <origin rpy="0 0 0"
@@ -44,7 +49,38 @@
   <joint name="trimble_joint" type="fixed" >
     <origin rpy="0 0 0"
-            xyz="1.81 0 1.5" />
+            xyz="0 0 -1.19" />
     <parent link="trimble"/>
     <child link="base_link"/>
+  </joint>
+  <joint name="imu_joint" type="fixed" >
+    <origin rpy="0 0 0"
+            xyz="0 0 0.15" />
+    <parent link="base_link"/>
+    <child link="imu"/>
+  </joint>
+  <!-- Radius of wheels 0.3 meters -->
+  <joint name="frwheel_joint" type="fixed" >
+    <origin rpy="0 0 0"
+            xyz="1 -0.75 0.165" />
+    <parent link="base_link"/>
+    <child link="frwheel"/>
+  </joint>
+  <joint name="flwheel_joint" type="fixed" >
+    <origin rpy="0 0 0"
+            xyz="1 0.75 0.165" />
+    <parent link="base_link"/>
+    <child link="flwheel"/>
+  </joint>
+  <joint name="rrwheel_joint" type="fixed" >
+    <origin rpy="0 0 0"
+            xyz="-1 -0.75 0.165" />
+    <parent link="base_link"/>
+    <child link="rrwheel"/>
+  </joint>
+  <joint name="rlwheel_joint" type="fixed" >
+    <origin rpy="0 0 0"
+            xyz="-1 0.75 0.165" />
+    <parent link="base_link"/>
+    <child link="rlwheel"/>
   </joint>
   <joint name="camera_left_joint" type="fixed" >

Commit message: Added trimble as its own link

File: rcv_description/urdf/rcv.xacro (robot description, xacro)
@@ -24,4 +24,10 @@
   <link name="left_optical"/>
   <link name="right_optical"/>
+  <joint name="trimble_joint" type="fixed" >
+    <origin rpy="0 0 0"
+            xyz="-1.81 0 -1.5" />
+    <parent link="trimble"/>
+    <child link="base_link"/>
+  </joint>
   <joint name="base_sensor_board_joint" type="fixed" >
     <origin rpy="0 0 0"
@@ -42,10 +48,4 @@
     <child link="velodyne_left"/>
   </joint>
-  <joint name="trimble_joint" type="fixed" >
-    <origin rpy="0 0 0"
-            xyz="0.06 0 0" />
-    <parent link="sensor_board_link"/>
-    <child link="trimble"/>
-  </joint>
   <joint name="camera_left_joint" type="fixed" >
     <origin rpy="0 0 0"

Commit message: Added the publishing of the mesh to the urdf instead of the script

File: rcv_description/urdf/rcv.xacro (robot description, xacro)
@@ -10,4 +10,10 @@
   <!-- Base link is the actual robot body, on the ground-->
   <link name="base_link">
+    <visual>
+      <origin rpy="0 0 3.14" xyz="0 0 0"/>
+        <geometry>
+          <mesh filename="package://rcv_description/meshes/RCV_assembly_stl_downsample.dae" scale="0.025 0.025 0.025"/>
+        </geometry>
+    </visual>
     <collision>
       <origin rpy="0 0 0" xyz="0 0 0.3"/>
@@ -31,5 +37,5 @@
   <joint name="trimble_joint" type="fixed" >
     <origin rpy="0 0 0"
-            xyz="-1.81 0 -1.5" />
+            xyz="0.09 0 -1.2" />
     <parent link="trimble"/>
     <child link="base_link"/>
@@ -37,5 +43,5 @@
   <joint name="base_sensor_board_joint" type="fixed" >
     <origin rpy="0 0 0"
-            xyz="1.75 0 1.5" />
+            xyz="-0.15 0 1.2" />
     <parent link="base_link"/>
     <child link="sensor_board_link"/>
